File: pcb/helios/fatboy-helios.kicad_pcb (KiCad board)
At the start: 2 copper layers, 232.2 x 108.2 mm, 76 parts, among them SW1 SW_Push, U1 Helios

Commit message: helios: use `libs/marbastlib` for symbols and footprints
Instead of implicitly relying on the assumption that the `marbastlib`
(or any other library, really) will be present in development
environment, expliciltly rely on the respective submodule version
of the library
Parts:
- MX1, MX10, MX11, MX12, MX13, MX14, MX15, MX16, MX17, MX18, MX19, MX2, MX20, MX21, MX22, MX23, MX24, MX25, MX26, MX27, MX28, MX29, MX3, MX30, MX31, MX32, MX33, MX34, MX35, MX36, MX4, MX5, MX6, MX7, MX8, MX9: footprint PCM_marbastlib-mx:SW_MX_HS_CPG151101S11_1u -> marbastlib-mx:SW_MX_HS_CPG151101S11_1u
- SW1: footprint PCM_marbastlib-various:SW_SKHLLCA010 -> marbastlib-various:SW_SKHLLCA010
Connections:
- U1 pad 32: unconnected-(U1-D+-Pad32) -> D+
- U1 pad 33: unconnected-(U1-D--Pad33) -> D-
